File: Hardware/ProtoSnap-LilyTwinkle.sch (EAGLE design)
At the start: 41 parts, among them U1 ATTINY85

Commit message: V10 commit; files as proposed for production. Changes: - BMASK added to programming vias - Pin numbers moved onto masked area on top side - Pin numbers added to bottom - Pin 1 marker added to programming header - Position of snapping holes tweaked slightly for durability improvement
Other:
- note added: "10"
- note removed: "01"
Changed lines of the file:
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@@
 <text x="164.846" y="113.03" size="2.1844" layer="91">3</text>
 <text x="172.72" y="7.62" size="3.81" layer="94">Team SparkFun</text>
-<text x="239.268" y="6.858" size="3.81" layer="94">01</text>
+<text x="239.268" y="6.858" size="3.81" layer="94">10</text>
 </plain>
 <instances>
